File: bkm-129x-simple-scart.kicad_pcb (KiCad board)
At the start: 2 copper layers, 105 x 89.3 mm, 51 parts, among them J1 SCART-F, J2 LEFT, J3 RIGHT, J5 Conn_02x32_Row_Letter_Last, Q1 DTC144EKA, SW1 LC2259EENP, U1 ADG1611, U2 THS7374, U3 arduino-nano-v3, U4 74LVC125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

Commit message: Revision B
Connections:
- U2 pad 9: GND -> +3V3
Routing:
- net GND: track 10.7 -> 9.43 mm, vias 8 -> 7
- net +3V3: track 16.0 -> 16.7 mm
Other:
- rule pad_to_mask_clearance: 0.2 -> 0
- board text added: "Rev. B"
- board text removed: "Rev. A"
